File: Kicad/Linear_Acuator_Control/Linear_Acuator_Control.kicad_sch (KiCad schematic)
At the start: 10 parts, among them K1 RT42xAxx, K3 RT42xAxx, Q1 IRLZ44N, Q2 IRLZ44N, U1 ESP32-S3-WROOM

Commit message: Rerouting dodgy traces, fixing ESP32 footprint
Connections:
- net +3V3: no longer names the net of U1.1 (3V3), U1.2 (3V3)
Changed lines of the file:
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@@
-	)
-	(symbol
-		(lib_id "power:+3V3")
-		(at 82.55 48.26 0)
-		(unit 1)
-		(exclude_from_sim no)
-		(in_bom yes)
-		(on_board yes)
-		(dnp no)
-		(fields_autoplaced yes)
-		(property "Reference" "#PWR07"
-			(at 82.55 52.07 0)
-			(effects
-				(font
-					(size 1.27 1.27)
-				)
-				(hide yes)
-			)
-		)
-		(property "Value" "+3V3"
-			(at 82.55 43.18 0)
-			(effects
-				(font
-					(size 1.27 1.27)
-				)
-			)
-		)
-		(property "Footprint" ""
-			(at 82.55 48.26 0)
-			(effects
-				(font
-					(size 1.27 1.27)
-				)
-				(hide yes)
-			)
-		)
-		(property "Datasheet" ""
-			(at 82.55 48.26 0)
-			(effects
-				(font
-					(size 1.27 1.27)
-				)
-				(hide yes)
-			)
-		)
-		(property "Description" "Power symbol creates a global label with name \"+3V3\""
-			(at 82.55 48.26 0)
-			(effects
-				(font
-					(size 1.27 1.27)
-				)
-				(hide yes)
-			)
-		)
-		(pin "1"
-		)
-		(instances
-			(project ""
-				(path "/f7047aaa-ba32-49d1-99b3-f492bbec601f"
-					(reference "#PWR07")
-					(unit 1)
-				)
-			)
-		)
 	)
 	(symbol
@@
 			)
 		)
-		(pin "24"
+		(pin "GND"
 		)
 		(pin "41"
@@
 		(pin "3"
 		)
-		(pin "23"
-		)
 		(pin "21"
 		)
-		(pin "44"
-		)
 		(pin "10"
 		)
@@
 		(pin "38"
 		)
-		(pin "22"
-		)
 		(pin "9"

Commit message: Changed Mosfets to better suit 3.3v logic levels
Parts:
- Q1, Q2: value IRLZ44N -> IRLB3813
Changed lines of the file:
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@@
 			)
 		)
-		(property "Value" "IRLZ44N"
+		(property "Value" "IRLB3813"
 			(at 191.77 91.4399 0)
 			(effects
@@
 			)
 		)
-		(property "Value" "IRLZ44N"
+		(property "Value" "IRLB3813"
 			(at 241.3 99.0599 0)
 			(effects
