File: Kicad/Linear_Acuator_Control/Linear_Acuator_Control.kicad_sch (KiCad schematic)
At the start: 20 parts, among them K1 RT42xAxx, K3 RT42xAxx, Q1 IRLB3813, Q2 IRLB3813, Q3 NMOS_Substrate, Q4 NMOS_Substrate, U1 ESP32-S3-WROOM

Commit message: finished routing with updated design
Parts:
- removed Q3, Q4: NMOS_Substrate, symbol Simulation_SPICE:NMOS_Substrate
- added Q3, Q5: 2N7002, Package_TO_SOT_SMD:SOT-23, symbol Transistor_FET:2N7002
Connections:
- net +24V: now also D4.1 (K)
- net GND: now also Q3.2 (S), Q5.2 (S)
- net at D3.2 (A), K3.A2: now also Q3.3 (D)
- net at R1.2, R2.1: now also Q3.1 (G)
- net at R3.2, R4.1: now also Q5.1 (G)
- net at D4.2 (A), K1.A2: now also Q5.3 (D)
Other:
- moved on the sheet: D4, R2, R4

Commit message: adding part numbers
for some reason the diodes dont work properly with lcsc idk will investigate
Parts:
- L1: value Linear_actuator -> Linear actuator 1
- L2: value Linear_actuator -> Linear Actuator 2
- L3: value Linear_actuator -> 24v 20A Input
- R1, R2: footprint Resistor_THT:R_Axial_DIN0207_L6.3mm_D2.5mm_P10.16mm_Horizontal -> Resistor_SMD:R_0603_1608Metric
- R3: value 1k -> 10k; footprint Resistor_THT:R_Axial_DIN0207_L6.3mm_D2.5mm_P10.16mm_Horizontal -> Resistor_SMD:R_0603_1608Metric
- R4: value 10k -> 1k; footprint Resistor_THT:R_Axial_DIN0207_L6.3mm_D2.5mm_P10.16mm_Horizontal -> Resistor_SMD:R_0603_1608Metric
- R5: footprint Resistor_THT:R_Axial_DIN0207_L6.3mm_D2.5mm_P10.16mm_Horizontal -> Resistor_SMD:R_0201_0603Metric
Connections:
- net Dir L1: now also U1.36 (GPIO39/MTCK); no longer R1.1
- net Dir L2: no longer R3.1
- net Speed L1: now also U1.39 (GPIO42/MTMS)
- net Net-(Q5-G): now reaches Q5.1 (G), R3.2, R4.1
- net Net-(Q5-G): now also R3.1
- net Net-(Q3-G): now reaches Q3.1 (G), R1.2, R2.1
- net Net-(Q3-G): now also R1.1
- net L1SwitchedLow: now reaches D1.2 (A), K3.11, Q1.2 (D)
